File: corne-wireless/corne-wireless.kicad_sch (KiCad schematic)
At the start: 90 parts, among them J2 OLED, J4 OLED, SW1 SW_PUSH, SW10 SW_PUSH, SW11 SW_PUSH, SW12 SW_PUSH, SW13 SW_PUSH, SW14 SW_PUSH, SW15 SW_PUSH, SW16 SW_PUSH, SW17 SW_PUSH, SW18 SW_PUSH, SW19 SW_PUSH, SW2 SW_PUSH, SW20 SW_PUSH, SW21 SW_PUSH, SW22 SW_PUSH, SW23 SW_PUSH, SW24 SW_PUSH, SW25 SW_PUSH, SW26 SW_PUSH, SW27 SW_PUSH, SW28 SW_PUSH, SW29 SW_PUSH, SW3 SW_PUSH, SW30 SW_PUSH, SW31 SW_PUSH, SW32 SW_PUSH, SW33 SW_PUSH, SW34 SW_PUSH, SW35 SW_PUSH, SW36 SW_PUSH, SW37 SW_PUSH, SW38 SW_PUSH, SW39 SW_PUSH, SW4 SW_PUSH, SW40 SW_PUSH, SW41 SW_PUSH, SW42 SW_PUSH, SW5 SW_PUSH, SW6 SW_PUSH, SW7 SW_PUSH, SW8 SW_PUSH, SW9 SW_PUSH, U1 ProMicro, U2 ProMicro

Commit message: Restart
Parts:
- removed D1, D10, D11, D12, D13, D14, D15, D16, D17, D18, D19, D2, D20, D21, D3, D4, D5, D6, D7, D8, D9: 1N4148, Diode_THT:D_DO-35_SOD27_P7.62mm_Horizontal, symbol Diode:1N4148
- added D1, D10, D11, D12, D14, D15, D16, D17, D18, D19, D2, D20, D21, D3, D4, D5, D6, D7, D8, D9: D, kbd:D3_SMD_v2, symbol Device:D
- added D13: D, kbd:D3_SMD_v2, symbol Diode:1N4148W
- added J1, J3: MJ-4PP-9, kbd:MJ-4PP-9_1side, symbol kbd:MJ-4PP-9
Connections:
- net GND1: now also J1.C
- net VCC: now also J1.D
- net data: now also J1.B
- net data_r: now also J3.B
- net row0: now also D6.1 (K)
- net row0_r: now also D27.1 (K)
- net row1: now also D12.1 (K)
- net row1_r: now also D33.1 (K)
- net row2: now also D18.1 (K)
- net row2_r: now also D39.1 (K)
- net row3: now also D21.1 (K)
- net row3_r: now also D42.1 (K)
- net at SW2.2: now also D2.2 (A)
- net at SW3.2: now also D3.2 (A)
- net at SW4.2: now also D4.2 (A)
- net at SW5.2: now also D5.2 (A)
- net at SW6.2: now also D6.2 (A)
- net at SW1.2: now also D1.2 (A)
- net at SW8.2: now also D8.2 (A)
- net at SW9.2: now also D9.2 (A)
- net at SW10.2: now also D10.2 (A)
- net at SW11.2: now also D11.2 (A)
- net at SW12.2: now also D12.2 (A)
- net at SW7.2: now also D7.2 (A)
- net at SW14.2: now also D14.2 (A)
- net at SW15.2: now also D15.2 (A)
- net at SW16.2: now also D16.2 (A)
- net at SW17.2: now also D17.2 (A)
- net at SW18.2: now also D18.2 (A)
- net at SW13.2: now also D13.2 (A)
- net at SW20.2: now also D20.2 (A)
- net at SW21.2: now also D21.2 (A)
- net at SW19.2: now also D19.2 (A)
- net at SW23.2: now also D23.2 (A)
- net at SW24.2: now also D24.2 (A)
- net at SW25.2: now also D25.2 (A)
- net at SW26.2: now also D26.2 (A)
- net at SW27.2: now also D27.2 (A)
- net at SW22.2: now also D22.2 (A)
- net at SW29.2: now also D29.2 (A)
- net at SW30.2: now also D30.2 (A)
- net at SW31.2: now also D31.2 (A)
- net at SW32.2: now also D32.2 (A)
- net at SW33.2: now also D33.2 (A)
- net at SW28.2: now also D28.2 (A)
- net at SW35.2: now also D35.2 (A)
- net at SW36.2: now also D36.2 (A)
- net at SW37.2: now also D37.2 (A)
- net at SW38.2: now also D38.2 (A)
- net at SW39.2: now also D39.2 (A)
- net at SW34.2: now also D34.2 (A)
- net at SW41.2: now also D41.2 (A)
- net at SW42.2: now also D42.2 (A)
- net at SW40.2: now also D40.2 (A)
- net VDD: no longer names the net of U2.21 (VCC)
- no-connect marks 10 -> 12
Other:
- moved on the sheet: RSW1, SW1, SW10, SW11, SW12, SW13, SW14, SW15, SW16, SW17, SW18, SW19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

Commit message: Prep for removal of OLED headers
Parts:
- removed J1, J3: MJ-4PP-9, kbd:MJ-4PP-9_1side, symbol kbd:MJ-4PP-9
- added J1, J2: Conn_01x02, symbol Connector_Generic:Conn_01x02
- added PMOS1, PMOS2: SSM3J328R, corne-wireless-fp:SOT-23F, symbol corne-wireless-sym:SSM3J328R
- added SW1, SW23: SW_SPDT, symbol Switch:SW_SPDT
- OL1: renamed from J2; symbol Connector_Generic:Conn_01x04 -> kbd:OLED
- OL2: renamed from J4; symbol Connector_Generic:Conn_01x04 -> kbd:OLED
- renumbered D4 to D10, D10 to D11, D16 to D12, D19 to D13, D5 to D14, D11 to D15, D17 to D16, D20 to D17, D6 to D18, D12 to D19, D7 to D2, D18 to D20, D28 to D23, D34 to D24, D23 to D25, D29 to D26, D35 to D27, D24 to D28, D30 to D29, D13 to D3, D36 to D30, D25 to D31, D31 to D32, D37 to D33, D40 to D34, D26 to D35, D32 to D36, D38 to D37, D41 to D38, D27 to D39, D2 to D4, D33 to D40, D39 to D41, D8 to D5, D14 to D6, D3 to D7, D9 to D8, D15 to D9, SW15 to SW10, SW4 to SW11, SW10 to SW12, SW16 to SW13, SW19 to SW14, SW5 to SW15, SW11 to SW16, SW20 to SW18, SW6 to SW19, SW1 to SW2, SW12 to SW20, SW18 to SW21, SW21 to SW22, SW22 to SW24, SW28 to SW25, SW34 to SW26, SW23 to SW27, SW29 to SW28, SW35 to SW29, SW7 to SW3, SW24 to SW30, SW30 to SW31, SW36 to SW32, SW25 to SW33, SW31 to SW34, SW37 to SW35, SW40 to SW36, SW26 to SW37, SW32 to SW38, SW38 to SW39, SW13 to SW4, SW41 to SW40, SW27 to SW41, SW33 to SW42, SW39 to SW43, SW42 to SW44, SW2 to SW5, SW8 to SW6, SW14 to SW7, SW3 to SW8
Connections:
- net GND1: now also OL1.4 (GND), J1.2 (Pin_2), PMOS1.1 (G)
- net SCL: now also OL1.2 (SCL)
- net SCL_r: now also OL2.2 (SCL)
- net SDA: now also OL1.1 (SDA)
- net SDA_r: now also OL2.1 (SDA)
- net VCC: now also OL1.3 (VCC)
- net row0: now also D1.1 (K), D10.1 (K), D14.1 (K), D4.1 (K), D7.1 (K)
- net row0_r: now also D22.1 (K), D25.1 (K), D28.1 (K), D31.1 (K), D35.1 (K)
- net row1: now also D11.1 (K), D15.1 (K), D2.1 (K), D5.1 (K), D8.1 (K)
- net row1_r: now also D23.1 (K), D26.1 (K), D29.1 (K), D32.1 (K), D36.1 (K)
- net row2: now also D12.1 (K), D16.1 (K), D3.1 (K), D6.1 (K), D9.1 (K)
- net row2_r: now also D24.1 (K), D27.1 (K), D30.1 (K), D33.1 (K), D37.1 (K)
- net row3: now also D13.1 (K), D17.1 (K)
- net row3_r: now also D34.1 (K), D38.1 (K)
- net battery+: now reaches U1.24 (RAW)
- net battery+: now also SW1.1 (A)
- net VDD: now reaches U2.21 (VCC)
- net VDD: now also OL2.3 (VCC)
- net GND2: now reaches U2.23 (GND)
- net GND2: now also OL2.4 (GND), RSW2.2, U2.3 (GND), U2.4 (GND), J2.2 (Pin_2), PMOS2.1 (G)
- net battery+_r: now reaches U2.24 (RAW)
- net battery+_r: now also SW23.1 (A)
- net LED: no longer names the net of U1.1 (TX0/D3)
- net LED_r: no longer names the net of U2.1 (TX0/D3)
- net data: no longer names the net of U1.2 (RX1/D2)
- net data_r: no longer names the net of U2.2 (RX1/D2)
- new net: PMOS1.2 (S), SW1.2 (B)
- new net: J1.1 (Pin_1), PMOS1.3 (D)
- new net: PMOS2.2 (S), SW23.2 (B)
- new net: J2.1 (Pin_1), PMOS2.3 (D)
- no-connect marks 12 -> 14
Other:
- moved on the sheet: D1, D10, D11, D12, D13, D14, D15, D16, D17, D18, D19, D2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

Commit message: Finalize PCB
Parts:
- removed OL1, OL2: OLED, kbd:OLED_1side, symbol kbd:OLED
- J1, J2: footprint (none) -> Connector_JST:JST_SH_BM02B-SRSS-TB_1x02-1MP_P1.00mm_Vertical
- SW1, SW23: footprint (none) -> Button_Switch_SMD:SW_SPDT_PCM12
Connections:
- net battery+: now also SW1.3 (C); no longer SW1.1 (A)
Other:
- moved on the sheet: J1, J2, PMOS1, PMOS2, RSW1, RSW2, SW1, SW23

Commit message: Change JST SH connector to PH
Parts:
- J1, J2: footprint Connector_JST:JST_SH_BM02B-SRSS-TB_1x02-1MP_P1.00mm_Vertical -> Connector_JST:JST_PH_B2B-PH-K_1x02_P2.00mm_Vertical
Changed lines of the file:
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@@
       (effects (font (size 1.27 1.27)))
     )
-    (property "Footprint" "Connector_JST:JST_SH_BM02B-SRSS-TB_1x02-1MP_P1.00mm_Vertical" (at 39.37 102.87 0)
+    (property "Footprint" "Connector_JST:JST_PH_B2B-PH-K_1x02_P2.00mm_Vertical" (at 39.37 102.87 0)
       (effects (font (size 1.27 1.27)) hide)
     )
@@
       (effects (font (size 1.27 1.27)))
     )
-    (property "Footprint" "Connector_JST:JST_SH_BM02B-SRSS-TB_1x02-1MP_P1.00mm_Vertical" (at 229.87 102.87 0)
+    (property "Footprint" "Connector_JST:JST_PH_B2B-PH-K_1x02_P2.00mm_Vertical" (at 229.87 102.87 0)
       (effects (font (size 1.27 1.27)) hide)
     )
